Commit message: Change urdf

File: src/robot_description/description/robot_core.xacro (robot description, xacro)
@@ -3,4 +3,7 @@
     <material name="white">
         <color rgba="1 1 1 1" />
+    </material>
+    <material name="red">
+        <color rgba="1 0 0 1" />
     </material>
     <material name="orange">

File: src/robot_description/description/robotic_arm.xacro (robot description, xacro)
@@ -1,13 +1,4 @@
 <?xml version="1.0"?>
 <robot xmlns:xacro="http://www.ros.org/wiki/xacro" >
-    <!-- <material name="red">
-        <color rgba="1 0 0 1"/>
-    </material>
-    <material name="blue">
-        <color rgba="0 0 1 1"/>
-    </material>
-    <material name="green">
-        <color rgba="0 0 0 1"/>
-    </material> -->
     <xacro:property name="box_x" value="0.3"/>
     <xacro:property name="box_y" value="0.2"/>
@@ -198,5 +189,5 @@
     </joint>
    <link name="link_four">
-        <xacro:property name="l4_box_width" value= "0.05"/>
+        <xacro:property name="l4_box_width" value= "0.06"/>
         <xacro:property name="l4_box_depth" value="0.07" />
         <xacro:property name="l4_box_height" value="${link_one_base_length / 2.0}" />

Commit message: Fixed Robotic arm appearance in gazebo world

File: src/robot_description/description/robot_core.xacro (robot description, xacro)
@@ -3,7 +3,4 @@
     <material name="white">
         <color rgba="1 1 1 1" />
-    </material>
-    <material name="red">
-        <color rgba="1 0 0 1" />
     </material>
     <material name="orange">

File: src/robot_description/description/robotic_arm.xacro (robot description, xacro)
@@ -44,13 +44,7 @@
         </collision>
         <inertial>
-            <origin xyz="0 0 0" rpy="0 0 0"/>
-            <mass value="${link_one_mass}"/>
-            <inertia
-                ixx="${(1/12) * link_one_mass * (3 * link_one_base_radius**2 + link_one_base_length**2)}"
-                ixy="0.0"
-                ixz="0.0"
-                iyy="${(1/12) * link_one_mass * (3 * link_one_base_radius**2 + link_one_base_length**2)}"
-                iyz="0.0"
-                izz="${(1/2) * link_one_mass * link_one_base_radius**2}"/>
+            <origin xyz="0 0 0.1" rpy="0 0 0"/> <!-- Adjust Z to center of link -->
+            <mass value="0.1"/>
+            <inertia ixx="0.001" ixy="0" ixz="0" iyy="0.001" iyz="0" izz="0.001"/>
         </inertial>
     </link>
@@ -74,13 +68,7 @@
         </collision>
         <inertial>
-            <origin xyz="0 0 0" rpy="0 0 0"/>
-            <mass value="${holder_mass}"/>
-            <inertia
-                ixx="${(1/12) * holder_mass * (holder_y*holder_y + holder_z*holder_z)}"
-                ixy="0.0"
-                ixz="0.0"
-                iyy="${(1/12) * holder_mass * (holder_x*holder_x + holder_z*holder_z)}"
-                iyz="0.0"
-                izz="${(1/12) * holder_mass * (holder_x*holder_x + holder_y*holder_y)}"/>
+            <origin xyz="0 0 0.1" rpy="0 0 0"/>
+            <mass value="0.1"/>
+            <inertia ixx="0.001" ixy="0" ixz="0" iyy="0.001" iyz="0" izz="0.001"/>
         </inertial>
     </link>
@@ -99,13 +87,7 @@
         </collision>
         <inertial>
-            <origin xyz="0 0 0" rpy="0 0 0"/>
-            <mass value="${holder_mass}"/>
-            <inertia
-                ixx="${(1/12) * holder_mass * (holder_y*holder_y + holder_z*holder_z)}"
-                ixy="0.0"
-                ixz="0.0"
-                iyy="${(1/12) * holder_mass * (holder_x*holder_x + holder_z*holder_z)}"
-                iyz="0.0"
-                izz="${(1/12) * holder_mass * (holder_x*holder_x + holder_y*holder_y)}"/>
+            <origin xyz="0 0 0.1" rpy="0 0 0"/> <!-- Adjust Z to center of link -->
+            <mass value="0.1"/>
+            <inertia ixx="0.001" ixy="0" ixz="0" iyy="0.001" iyz="0" izz="0.001"/>
         </inertial>
     </link>
@@ -136,13 +118,7 @@
         </collision>
         <inertial>
-            <origin xyz="0 0 ${link_two_length/2}" rpy="0 0 0"/>
-            <mass value="${link_two_mass}"/>
-            <inertia
-                ixx="${(1/12) * link_two_mass * (link_two_thickness*link_two_thickness + link_two_length*link_two_length)}"
-                ixy="0.0"
-                ixz="0.0"
-                iyy="${(1/12) * link_two_mass * (link_two_width*link_two_width + link_two_length*link_two_length)}"
-                iyz="0.0"
-                izz="${(1/12) * link_two_mass * (link_two_width*link_two_width + link_two_thickness*link_two_thickness)}"/>
+            <origin xyz="0 0 0.1" rpy="0 0 0"/> <!-- Adjust Z to center of link -->
+            <mass value="0.1"/>
+            <inertia ixx="0.001" ixy="0" ixz="0" iyy="0.001" iyz="0" izz="0.001"/>
         </inertial>
     </link>
@@ -170,13 +146,7 @@
         </collision>
         <inertial>
-            <origin xyz="0 0 ${link_three_length/2}" rpy="0 0 0"/>
-            <mass value="${link_three_mass}"/>
-            <inertia
-                ixx="${(1/12) * link_three_mass * (link_two_thickness*link_two_thickness + link_three_length*link_three_length)}"
-                ixy="0.0"
-                ixz="0.0"
-                iyy="${(1/12) * link_three_mass * (link_two_width*link_two_width + link_three_length*link_three_length)}"
-                iyz="0.0"
-                izz="${(1/12) * link_three_mass * (link_two_width*link_two_width + link_two_thickness*link_two_thickness)}"/>
+            <origin xyz="0 0 0.1" rpy="0 0 0"/> <!-- Adjust Z to center of link -->
+            <mass value="0.1"/>
+            <inertia ixx="0.001" ixy="0" ixz="0" iyy="0.001" iyz="0" izz="0.001"/>
         </inertial>
     </link>
@@ -206,12 +176,7 @@
         </collision>
         <inertial>
-            <origin xyz="0 0 0" rpy="0 0 0"/>
-            <mass value="${link_four_mass}"/>
-            <inertia
-                ixx="${(1/12) * link_four_mass * (l4_box_depth**2 + l4_box_height**2)}"
-                ixy="0.0" ixz="0.0"
-                iyy="${(1/12) * link_four_mass * (l4_box_width**2 + l4_box_height**2)}"
-                iyz="0.0"
-                izz="${(1/12) * link_four_mass * (l4_box_width**2 + l4_box_depth**2)}"/>
+            <origin xyz="0 0 0.1" rpy="0 0 0"/> <!-- Adjust Z to center of link -->
+            <mass value="0.1"/>
+            <inertia ixx="0.001" ixy="0" ixz="0" iyy="0.001" iyz="0" izz="0.001"/>
         </inertial>
     </link>
@@ -237,12 +202,7 @@
         </collision>
        <inertial>
-            <origin xyz="0 0 ${finger_length/2}" rpy="0 0 0"/>
-            <mass value="${finger_mass}"/>
-            <inertia
-                ixx="${(1/12) * finger_mass * (finger_thickness*finger_thickness + finger_length*finger_length)}"
-                ixy="0.0" ixz="0.0"
-                iyy="${(1/12) * finger_mass * (finger_width*finger_width + finger_length*finger_length)}"
-                iyz="0.0"
-                izz="${(1/12) * finger_mass * (finger_width*finger_width + finger_thickness*finger_thickness)}"/>
+            <origin xyz="0 0 0.1" rpy="0 0 0"/> <!-- Adjust Z to center of link -->
+            <mass value="0.1"/>
+            <inertia ixx="0.001" ixy="0" ixz="0" iyy="0.001" iyz="0" izz="0.001"/>
         </inertial>
     </link>
@@ -269,16 +229,11 @@
         </collision>
         <inertial>
-            <origin xyz="0 ${finger_width/2} ${finger_length/2}" rpy="0 0 0"/>
-            <mass value="${finger_mass}"/>
-            <inertia
-                ixx="${(1/12) * finger_mass * (finger_thickness*finger_thickness + finger_length*finger_length)}"
-                ixy="0.0" ixz="0.0"
-                iyy="${(1/12) * finger_mass * (finger_width*finger_width + finger_length*finger_length)}"
-                iyz="0.0"
-                izz="${(1/12) * finger_mass * (finger_width*finger_width + finger_thickness*finger_thickness)}"/>
+            <origin xyz="0 0 0.1" rpy="0 0 0"/> <!-- Adjust Z to center of link -->
+            <mass value="0.1"/>
+            <inertia ixx="0.001" ixy="0" ixz="0" iyy="0.001" iyz="0" izz="0.001"/>
         </inertial>
     </link>
     <joint name="right_finger_joint" type="prismatic">
-        <mimic joint="left_finger_joint" multiplier="-1.0" offset="0"/>
+        <!-- <mimic joint="left_finger_joint" multiplier="-1.0" offset="0"/>  -->
         <parent link="link_four"/>
         <child link="right_finger"/>
@@ -302,10 +257,8 @@
         </collision>
         <inertial>
-            <origin xyz="${0.01/2} ${0.01/2} 0" rpy="0 0 0" />
-            <mass value="0.01" />
-            <inertia ixx="0.000000167" ixy="0.0" ixz="0.0"
-                    iyy="0.000000167" iyz="0.0"
-                    izz="0.000000167" />
-    </inertial>
+            <origin xyz="0 0 0.1" rpy="0 0 0"/> <!-- Adjust Z to center of link -->
+            <mass value="0.1"/>
+            <inertia ixx="0.001" ixy="0" ixz="0" iyy="0.001" iyz="0" izz="0.001"/>
+        </inertial>
     </link>
     <joint name="camera_gripper_joint" type="fixed">
@@ -329,9 +282,7 @@
         </collision>
         <inertial>
-            <origin xyz="${0.01/2} ${0.01/2} 0" rpy="0 0 0" />
-            <mass value="0.01" />
-            <inertia ixx="0.000000167" ixy="0.0" ixz="0.0"
-                    iyy="0.000000167" iyz="0.0"
-                    izz="0.000000167" />
+            <origin xyz="0 0 0.1" rpy="0 0 0"/> <!-- Adjust Z to center of link -->
+            <mass value="0.1"/>
+            <inertia ixx="0.001" ixy="0" ixz="0" iyy="0.001" iyz="0" izz="0.001"/>
         </inertial>
     </link>
