Commit message: fix: map appears in rviz

File: src/robot_description/description/lidar.xacro (robot description, xacro)
@@ -15,5 +15,5 @@
         <collision>
             <geometry>
-                <cylinder radius="${lidar_radius}" length="${lidar_length}"/>
+                <cylinder radius="${lidar_radius}" length="${lidar_length/2}"/>
             </geometry>
         </collision>
@@ -40,5 +40,5 @@
             </scan>
             <range>
-                <min>0.0</min>
+                <min>0.12</min>
                 <max>12.0</max>
                 <resolution>0.01</resolution>

File: src/robot_description/description/robot.urdf.xacro (robot description, xacro)
@@ -13,4 +13,4 @@
     <xacro:include filename="camera.xacro"/>
     <xacro:include filename="imu.xacro"/>
-    <xacro:include filename="robotic_arm.xacro"/>
+    <!-- <xacro:include filename="robotic_arm.xacro"/> -->
 </robot>

File: src/robot_description/description/robotic_arm.xacro (robot description, xacro)
@@ -43,8 +43,14 @@
             <origin xyz="0 0 0" rpy="0 0 0"/>
         </collision>
-        <inertial>
-            <origin xyz="0 0 0.1" rpy="0 0 0"/> <!-- Adjust Z to center of link -->
+      <inertial>
+            <origin xyz="0 0 0" rpy="0 0 0"/>
             <mass value="0.1"/>
-            <inertia ixx="0.001" ixy="0" ixz="0" iyy="0.001" iyz="0" izz="0.001"/>
+            <inertia
+                ixx="${(1/12) * 0.1 * (3 * link_one_base_radius**2 + link_one_base_length**2)}"
+                ixy="0"
+                ixz="0"
+                iyy="${(1/12) * 0.1 * (3 * link_one_base_radius**2 + link_one_base_length**2)}"
+                iyz="0"
+                izz="${(1/2) * 0.1 * link_one_base_radius**2}"/>
         </inertial>
     </link>
@@ -68,7 +74,13 @@
         </collision>
         <inertial>
-            <origin xyz="0 0 0.1" rpy="0 0 0"/>
+            <origin xyz="0 0 0" rpy="0 0 0"/>
             <mass value="0.1"/>
-            <inertia ixx="0.001" ixy="0" ixz="0" iyy="0.001" iyz="0" izz="0.001"/>
+            <inertia
+                ixx="${(1/12) * 0.1 * (holder_y**2 + holder_z**2)}"
+                ixy="0"
+                ixz="0"
+                iyy="${(1/12) * 0.1 * (holder_x**2 + holder_z**2)}"
+                iyz="0"
+                izz="${(1/12) * 0.1 * (holder_x**2 + holder_y**2)}"/>
         </inertial>
     </link>
@@ -87,7 +99,13 @@
         </collision>
         <inertial>
-            <origin xyz="0 0 0.1" rpy="0 0 0"/> <!-- Adjust Z to center of link -->
-            <mass value="0.1"/>
-            <inertia ixx="0.001" ixy="0" ixz="0" iyy="0.001" iyz="0" izz="0.001"/>
+            <origin xyz="0 0 0" rpy="0 0 0"/>
+            <mass value="${holder_mass}"/>
+            <inertia
+                ixx="${(1/12) * holder_mass * (holder_y**2 + holder_z**2)}"
+                ixy="0"
+                ixz="0"
+                iyy="${(1/12) * holder_mass * (holder_x**2 + holder_z**2)}"
+                iyz="0"
+                izz="${(1/12) * holder_mass * (holder_x**2 + holder_y**2)}"/>
         </inertial>
     </link>
@@ -118,7 +136,13 @@
         </collision>
         <inertial>
-            <origin xyz="0 0 0.1" rpy="0 0 0"/> <!-- Adjust Z to center of link -->
-            <mass value="0.1"/>
-            <inertia ixx="0.001" ixy="0" ixz="0" iyy="0.001" iyz="0" izz="0.001"/>
+            <origin xyz="0 0 ${link_two_length/2}" rpy="0 0 0"/>
+            <mass value="${link_two_mass}"/>
+            <inertia
+                ixx="${(1/12) * link_two_mass * (link_two_thickness**2 + link_two_length**2)}"
+                ixy="0"
+                ixz="0"
+                iyy="${(1/12) * link_two_mass * (link_two_width**2 + link_two_length**2)}"
+                iyz="0"
+                izz="${(1/12) * link_two_mass * (link_two_width**2 + link_two_thickness**2)}"/>
         </inertial>
     </link>
@@ -146,7 +170,13 @@
         </collision>
         <inertial>
-            <origin xyz="0 0 0.1" rpy="0 0 0"/> <!-- Adjust Z to center of link -->
-            <mass value="0.1"/>
-            <inertia ixx="0.001" ixy="0" ixz="0" iyy="0.001" iyz="0" izz="0.001"/>
+            <origin xyz="0 0 ${link_three_length/2}" rpy="0 0 0"/>
+            <mass value="${link_three_mass}"/>
+            <inertia
+                ixx="${(1/12) * link_three_mass * (link_two_thickness**2 + link_three_length**2)}"
+                ixy="0"
+                ixz="0"
+                iyy="${(1/12) * link_three_mass * (link_two_width**2 + link_three_length**2)}"
+                iyz="0"
+                izz="${(1/12) * link_three_mass * (link_two_width**2 + link_two_thickness**2)}"/>
         </inertial>
     </link>
@@ -176,7 +206,13 @@
         </collision>
         <inertial>
-            <origin xyz="0 0 0.1" rpy="0 0 0"/> <!-- Adjust Z to center of link -->
-            <mass value="0.1"/>
-            <inertia ixx="0.001" ixy="0" ixz="0" iyy="0.001" iyz="0" izz="0.001"/>
+            <origin xyz="0 0 0" rpy="0 0 0"/>
+            <mass value="${link_four_mass}"/>
+            <inertia
+                ixx="${(1/12) * link_four_mass * (l4_box_depth**2 + l4_box_height**2)}"
+                ixy="0"
+                ixz="0"
+                iyy="${(1/12) * link_four_mass * (l4_box_width**2 + l4_box_height**2)}"
+                iyz="0"
+                izz="${(1/12) * link_four_mass * (l4_box_width**2 + l4_box_depth**2)}"/>
         </inertial>
     </link>
@@ -202,7 +238,13 @@
         </collision>
        <inertial>
-            <origin xyz="0 0 0.1" rpy="0 0 0"/> <!-- Adjust Z to center of link -->
-            <mass value="0.1"/>
-            <inertia ixx="0.001" ixy="0" ixz="0" iyy="0.001" iyz="0" izz="0.001"/>
+            <origin xyz="0 0 ${finger_length/2}" rpy="0 0 0"/>
+            <mass value="${finger_mass}"/>
+            <inertia
+                ixx="${(1/12) * finger_mass * (finger_thickness**2 + finger_length**2)}"
+                ixy="0"
+                ixz="0"
+                iyy="${(1/12) * finger_mass * (finger_width**2 + finger_length**2)}"
+                iyz="0"
+                izz="${(1/12) * finger_mass * (finger_width**2 + finger_thickness**2)}"/>
         </inertial>
     </link>
@@ -229,7 +271,13 @@
         </collision>
         <inertial>
-            <origin xyz="0 0 0.1" rpy="0 0 0"/> <!-- Adjust Z to center of link -->
-            <mass value="0.1"/>
-            <inertia ixx="0.001" ixy="0" ixz="0" iyy="0.001" iyz="0" izz="0.001"/>
+            <origin xyz="0 ${finger_width/2} ${finger_length/2}" rpy="0 0 0"/>
+            <mass value="${finger_mass}"/>
+            <inertia
+                ixx="${(1/12) * finger_mass * (finger_thickness**2 + finger_length**2)}"
+                ixy="0"
+                ixz="0"
+                iyy="${(1/12) * finger_mass * (finger_width**2 + finger_length**2)}"
+                iyz="0"
+                izz="${(1/12) * finger_mass * (finger_width**2 + finger_thickness**2)}"/>
         </inertial>
     </link>

File: src/robot_description/description/ros2_control.xacro (robot description, xacro)
@@ -53,5 +53,5 @@
             </joint>
             <!-- For Arm -->
-            <joint name="link_one_joint">
+            <!-- <joint name="link_one_joint">
                 <command_interface name="position"/>
                 <state_interface name="position"/>
@@ -67,5 +67,5 @@
                 <state_interface name="position"/>
                 <state_interface name="velocity"/>
-            </joint>
+            </joint> -->
         </ros2_control>
     </xacro:if>
